File: non-contact-sensor/non-contact-sensor.sch (KiCad schematic (older format))
At the start: 19 parts, among them J1 Conn_01x02, Q1 2N3904, U1 4011, U2 4011, U3 74LVC

Commit message: Added a parts list, updated with parts for non-contact AC voltage sensor. Started work on front-end circuit, which will be used for controlling both input from manual buttons and a monochrome eInk screen.
Parts:
- D1, D2: footprint Diode_SMD:D_0603_1608Metric -> Diode_SMD:D_SOD-323
Changed lines of the file:
@@
 F 0 "D1" V 1904 3779 50  0000 L CNN
 F 1 "1N4148" V 1995 3779 50  0000 L CNN
-F 2 "Diode_SMD:D_0603_1608Metric" H 1950 3525 50  0001 C CNN
+F 2 "Diode_SMD:D_SOD-323" H 1950 3525 50  0001 C CNN
 F 3 "https://assets.nexperia.com/documents/data-sheet/1N4148_1N4448.pdf" H 1950 3700 50  0001 C CNN
 	1    1950 3700
@@
 F 0 "D2" H 6100 3134 50  0000 C CNN
 F 1 "1N4148" H 6100 3225 50  0000 C CNN
-F 2 "Diode_SMD:D_0603_1608Metric" H 6100 3175 50  0001 C CNN
+F 2 "Diode_SMD:D_SOD-323" H 6100 3175 50  0001 C CNN
 F 3 "https://assets.nexperia.com/documents/data-sheet/1N4148_1N4448.pdf" H 6100 3350 50  0001 C CNN
 	1    6100 3350
